Commit message: validated PID and integration, still needs to fix urdf links

File: ros2_ws/src/gazebo_mujoco_bridge/urdf/so101.urdf (robot description, URDF)
Before this commit: robot so101, 7 links, 6 joints
Links:
- added link world
- link base_link: geometry collision mesh filename=package://gazebo_mujoco_bridge/meshes/base_motor_holder_so1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; collision mesh filename=package://gazebo_mujoco_bridge/meshes/base_so101_v2.stl
Joints:
- added joint base_fixed_to_world: type fixed, parent world, child base_link, origin xyz=0 0 0 rpy=0 0 0

File: ros2_ws/src/gazebo_mujoco_bridge/urdf/so101.urdf.xacro (robot description, xacro)
@@ -3,5 +3,4 @@
   <!-- Override mesh_dir to point to your STL assets -->
   <xacro:arg name="mesh_dir" default="package://gazebo_mujoco_bridge/meshes"/>
-       xmlns:xacro="http://www.ros.org/wiki/xacro">
   <!-- ═══════════ Gazebo plugins ═══════════ -->
   <!-- JointPositionController for each joint -->
@@ -65,4 +64,10 @@
   </gazebo>
   <!-- ═══════════ Links & Joints ═══════════ -->
+  <link name="world"/>
+  <joint name="base_fixed_to_world" type="fixed">
+    <parent link="world"/>
+    <child link="base_link"/>
+    <origin xyz="0 0 0" rpy="0 0 0"/>
+  </joint>
   <link name="base_link">
     <inertial>
@@ -71,4 +76,16 @@
       <inertia ixx="0.00013613" ixy="0.00000000" ixz="0.00000000" iyy="0.00013181" iyz="0.00000000" izz="0.00011323"/>
     </inertial>
+    <collision name="base_link_collision_0">
+      <origin xyz="-0.00636471 -0.00009944 -0.00240000" rpy="1.57079633 -0.00000000 1.57079633"/>
+      <geometry>
+        <mesh filename="package://gazebo_mujoco_bridge/meshes/base_motor_holder_so101_v1.stl"/>
+      </geometry>
+    </collision>
+    <collision name="base_link_collision_1">
+      <origin xyz="-0.00636471 -0.00000001 -0.00240000" rpy="1.57079633 -0.00000000 1.57079633"/>
+      <geometry>
+        <mesh filename="package://gazebo_mujoco_bridge/meshes/base_so101_v2.stl"/>
+      </geometry>
+    </collision>
   </link>
   <link name="shoulder_link">

File: simulation_code/model/so101.urdf.xacro (robot description, xacro)
@@ -3,5 +3,4 @@
   <!-- Override mesh_dir to point to your STL assets -->
   <xacro:arg name="mesh_dir" default="package://gazebo_mujoco_bridge/meshes"/>
-       xmlns:xacro="http://www.ros.org/wiki/xacro">
   <!-- ═══════════ Gazebo plugins ═══════════ -->
   <!-- JointPositionController for each joint -->
@@ -65,4 +64,10 @@
   </gazebo>
   <!-- ═══════════ Links & Joints ═══════════ -->
+  <link name="world"/>
+  <joint name="base_fixed_to_world" type="fixed">
+    <parent link="world"/>
+    <child link="base_link"/>
+    <origin xyz="0 0 0" rpy="0 0 0"/>
+  </joint>
   <link name="base_link">
     <inertial>
@@ -107,4 +112,28 @@
       </material>
     </visual>
+    <collision name="base_link_collision_0">
+      <origin xyz="-0.00636471 -0.00009944 -0.00240000" rpy="1.57079633 -0.00000000 1.57079633"/>
+      <geometry>
+        <mesh filename="package://gazebo_mujoco_bridge/meshes/base_motor_holder_so101_v1.stl"/>
+      </geometry>
+    </collision>
+    <collision name="base_link_collision_1">
+      <origin xyz="-0.00636471 -0.00000001 -0.00240000" rpy="1.57079633 -0.00000000 1.57079633"/>
+      <geometry>
+        <mesh filename="package://gazebo_mujoco_bridge/meshes/base_so101_v2.stl"/>
+      </geometry>
+    </collision>
+    <collision name="base_link_collision_2">
+      <origin xyz="0.02633530 -0.00000001 0.04370000" rpy="-0.00000000 -0.00000000 0.00000000"/>
+      <geometry>
+        <mesh filename="package://gazebo_mujoco_bridge/meshes/sts3215_03a_v1.stl"/>
+      </geometry>
+    </collision>
+    <collision name="base_link_collision_3">
+      <origin xyz="-0.03098270 -0.00019944 0.04740000" rpy="1.57079633 -0.00000000 1.57079633"/>
+      <geometry>
+        <mesh filename="package://gazebo_mujoco_bridge/meshes/waveshare_mounting_plate_so101_v2.stl"/>
+      </geometry>
+    </collision>
   </link>
   <link name="shoulder_link">

Commit message: Fixed the so101 model in gazebo

File: ros2_ws/src/gazebo_mujoco_bridge/urdf/so101.urdf (robot description, URDF)
Before this commit: robot so101, 8 links, 7 joints
Joints:
- joint shoulder_lift: origin xyz=-0.03039920 -0.01827780 -0.05420000 rpy=0.00000000 -1.57079633 1.57079633 -> xyz=-0.03039920 -0.01827780 -0.05420000 rpy=0.00000000 -1.57079633 -1.57079633

File: simulation_code/model/so101.urdf.xacro (robot description, xacro)
@@ -74,5 +74,5 @@
       <origin xyz="0.01371790 -0.00005197 0.03348430" rpy="0 0 0"/>
       <mass value="0.14700000"/>
-      <inertia ixx="0.00013613" ixy="0.00000000" ixz="0.00000000" iyy="0.00013181" iyz="0.00000000" izz="0.00011323"/>
+      <inertia ixx="0.00011469" ixy="-0.00000046" ixz="0.00000497" iyy="0.00013612" iyz="0.00000010" izz="0.00013036"/>
     </inertial>
     <visual name="base_link_visual_0">
@@ -141,5 +141,5 @@
       <origin xyz="-0.03076040 -0.00001667 -0.02527130" rpy="0 0 0"/>
       <mass value="0.10000600"/>
-      <inertia ixx="0.00008378" ixy="0.00000000" ixz="0.00000000" iyy="0.00008104" iyz="0.00000000" izz="0.00002396"/>
+      <inertia ixx="0.00008376" ixy="0.00000008" ixz="-0.00000116" iyy="0.00008104" iyz="0.00000015" izz="0.00002398"/>
     </inertial>
     <visual name="shoulder_link_visual_0">
@@ -201,5 +201,5 @@
       <origin xyz="-0.08984710 -0.00838224 0.01840890" rpy="0 0 0"/>
       <mass value="0.10300000"/>
-      <inertia ixx="0.00015087" ixy="0.00000000" ixz="0.00000000" iyy="0.00014249" iyz="0.00000000" izz="0.00003725"/>
+      <inertia ixx="0.00004080" ixy="-0.00001978" ixz="-0.00000004" iyy="0.00014732" iyz="0.00000001" izz="0.00014249"/>
     </inertial>
     <visual name="upper_arm_link_visual_0">
@@ -246,5 +246,5 @@
       <origin xyz="-0.09807010 0.00324376 0.01828310" rpy="0 0 0"/>
       <mass value="0.10400000"/>
-      <inertia ixx="0.00016026" ixy="0.00000000" ixz="0.00000000" iyy="0.00014530" iyz="0.00000000" izz="0.00002831"/>
+      <inertia ixx="0.00002874" ixy="0.00000741" ixz="0.00000126" iyy="0.00015984" iyz="-0.00000005" izz="0.00014529"/>
     </inertial>
     <visual name="lower_arm_link_visual_0">
@@ -306,5 +306,5 @@
       <origin xyz="-0.00010331 -0.03861430 0.02811560" rpy="0 0 0"/>
       <mass value="0.07900000"/>
-      <inertia ixx="0.00003683" ixy="0.00000000" ixz="0.00000000" iyy="0.00002745" iyz="0.00000000" izz="0.00001894"/>
+      <inertia ixx="0.00003683" ixy="0.00000002" ixz="-0.00000005" iyy="0.00002539" iyz="0.00000364" izz="0.00002100"/>
     </inertial>
     <visual name="wrist_link_visual_0">
@@ -351,5 +351,5 @@
       <origin xyz="0.00021363 0.00024514 -0.02518700" rpy="0 0 0"/>
       <mass value="0.08700000"/>
-      <inertia ixx="0.00004337" ixy="0.00000000" ixz="0.00000000" iyy="0.00003772" iyz="0.00000000" izz="0.00002428"/>
+      <inertia ixx="0.00002751" ixy="-0.00000034" ixz="-0.00000574" iyy="0.00004337" iyz="-0.00000005" izz="0.00003451"/>
     </inertial>
     <visual name="gripper_link_visual_0">
@@ -396,5 +396,5 @@
       <origin xyz="-0.00157495 -0.03002440 0.01927550" rpy="0 0 0"/>
       <mass value="0.01200000"/>
-      <inertia ixx="0.00000664" ixy="0.00000000" ixz="0.00000000" iyy="0.00000529" iyz="0.00000000" izz="0.00000187"/>
+      <inertia ixx="0.00000661" ixy="-0.00000032" ixz="-0.00000001" iyy="0.00000189" iyz="-0.00000011" izz="0.00000529"/>
     </inertial>
     <visual name="moving_jaw_link_visual_0">
